Commit message: Add camera and depth camera configurations to URDF

File: sawyer_description/urdf/sawyer.urdf.xacro (robot description, xacro)
@@ -22,3 +22,89 @@
   </xacro:include>
   </xacro:if>
+  <joint name="camera_joint" type="fixed">
+    <parent link="base"/>
+    <child link="camera_link"/>
+    <origin xyz="0.305 0 0.08" rpy="0 0 0"/>
+</joint>
+<link name="camera_link">
+    <visual>
+        <geometry>
+            <box size="0.010 0.03 0.03"/>
+        </geometry>
+        <material name="red"/>
+    </visual>
+</link>
+<joint name="camera_optical_joint" type="fixed">
+    <parent link="camera_link"/>
+    <child link="camera_link_optical"/>
+    <origin xyz="0 0 0" rpy="${-pi/2} 0 ${-pi/2}"/>
+</joint>
+<link name="camera_link_optical"></link>
+<gazebo reference="camera_link">
+    <material>Gazebo/Red</material>
+    <sensor name="camera" type="camera">
+        <pose> 0 0 0 0 0 0 </pose>
+        <visualize>true</visualize>
+        <update_rate>10</update_rate>
+        <camera>
+            <horizontal_fov>1.089</horizontal_fov>
+            <image>
+                <format>R8G8B8</format>
+                <width>640</width>
+                <height>480</height>
+            </image>
+            <clip>
+                <near>0.05</near>
+                <far>8.0</far>
+            </clip>
+        </camera>
+        <plugin name="camera_controller" filename="libgazebo_ros_camera.so">
+            <frame_name>camera_link_optical</frame_name>
+        </plugin>
+    </sensor>
+</gazebo>
+<joint name="depth_camera_joint" type="fixed">
+  <parent link="base"/>
+  <child link="depth_camera_link"/>
+  <origin xyz="0.305 0.1 0.08" rpy="0 0 0"/>
+</joint>
+<link name="depth_camera_link">
+  <visual>
+    <geometry>
+      <box size="0.010 0.03 0.03"/>
+    </geometry>
+    <material name="blue"/>
+  </visual>
+</link>
+<joint name="depth_camera_optical_joint" type="fixed">
+  <parent link="depth_camera_link"/>
+  <child link="depth_camera_link_optical"/>
+  <origin xyz="0 0 0" rpy="${-pi/2} 0 ${-pi/2}"/>
+</joint>
+<link name="depth_camera_link_optical"/>
+<gazebo reference="depth_camera_link">
+  <material>Gazebo/Blue</material>
+  <sensor name="depth_camera" type="depth">
+    <pose>0 0 0 0 0 0</pose>
+    <visualize>true</visualize>
+    <update_rate>10</update_rate>
+    <camera>
+      <horizontal_fov>1.047</horizontal_fov>
+      <image>
+        <format>R8G8B8</format>
+        <width>640</width>
+        <height>480</height>
+      </image>
+      <clip>
+        <near>0.05</near>
+        <far>8.0</far>
+      </clip>
+    </camera>
+    <plugin name="depth_camera_controller" filename="libgazebo_ros_depth_camera.so">
+      <frame_name>depth_camera_link_optical</frame_name>
+      <min_depth>0.05</min_depth>
+      <max_depth>8.0</max_depth>
+    </plugin>
+  </sensor>
+</gazebo>
 </robot>

Commit message: Update camera joint position and comment out depth camera joint in URDF

File: sawyer_description/urdf/sawyer.urdf.xacro (robot description, xacro)
@@ -25,5 +25,5 @@
     <parent link="base"/>
     <child link="camera_link"/>
-    <origin xyz="0.305 0 0.08" rpy="0 0 0"/>
+    <origin xyz="1.5 0 1.25" rpy="0 1.57079632679 0"/>
 </joint>
 <link name="camera_link">
@@ -64,4 +64,5 @@
     </sensor>
 </gazebo>
+<!--
 <joint name="depth_camera_joint" type="fixed">
   <parent link="base"/>
@@ -107,4 +108,4 @@
     </plugin>
   </sensor>
-</gazebo>
+</gazebo> -->
 </robot>

Commit message: Add RGB and depth camera configurations to URDF

File: sawyer_description/urdf/sawyer.urdf.xacro (robot description, xacro)
@@ -5,5 +5,7 @@
   <xacro:arg name="static" default="true"/>
   <xacro:arg name="electric_gripper" default="false"/>
-  <!-- Sawyer Base URDF -->
+  <!-- ======================= -->
+  <!-- SAWYER BASE -->
+  <!-- ======================= -->
   <xacro:include filename="$(find sawyer_description)/urdf/sawyer_base.urdf.xacro">
     <xacro:arg name="gazebo" value="${gazebo}"/>
@@ -11,100 +13,117 @@
   </xacro:include>
   <xacro:if value="$(arg gazebo)">
-  <xacro:include filename="$(find sawyer_description)/urdf/sawyer_base.gazebo.xacro">
-    <xacro:arg name="static" value="${static}"/>
-    <xacro:arg name="pedestal" value="${pedestal}"/>
-  </xacro:include>
+    <xacro:include filename="$(find sawyer_description)/urdf/sawyer_base.gazebo.xacro">
+      <xacro:arg name="static" value="${static}"/>
+      <xacro:arg name="pedestal" value="${pedestal}"/>
+    </xacro:include>
   </xacro:if>
-  <!-- Electric Gripper End Effector -->
   <xacro:if value="$(arg electric_gripper)">
-  <xacro:include filename="$(find sawyer_description)/urdf/sawyer_electric_gripper.urdf.xacro">
-    <xacro:arg name="gazebo" value="${gazebo}"/>
-  </xacro:include>
+    <xacro:include filename="$(find sawyer_description)/urdf/sawyer_electric_gripper.urdf.xacro">
+      <xacro:arg name="gazebo" value="${gazebo}"/>
+    </xacro:include>
   </xacro:if>
+  <!-- ======================= -->
+  <!-- RGB CAMERA -->
+  <!-- ======================= -->
   <joint name="camera_joint" type="fixed">
     <parent link="base"/>
     <child link="camera_link"/>
-    <origin xyz="0.305 0 0.08" rpy="0 0 0"/>
-</joint>
-<link name="camera_link">
+    <origin xyz="1.5 0 1.25" rpy="0 1.57079632679 0"/>
+  </joint>
+  <link name="camera_link">
     <visual>
-        <geometry>
-            <box size="0.010 0.03 0.03"/>
-        </geometry>
-        <material name="red"/>
+      <geometry>
+        <box size="0.010 0.03 0.03"/>
+      </geometry>
+      <material name="red"/>
     </visual>
-</link>
-<joint name="camera_optical_joint" type="fixed">
+  </link>
+  <joint name="camera_optical_joint" type="fixed">
     <parent link="camera_link"/>
     <child link="camera_link_optical"/>
     <origin xyz="0 0 0" rpy="${-pi/2} 0 ${-pi/2}"/>
-</joint>
-<link name="camera_link_optical"></link>
-<gazebo reference="camera_link">
+  </joint>
+  <link name="camera_link_optical"/>
+  <gazebo reference="camera_link">
     <material>Gazebo/Red</material>
-    <sensor name="camera" type="camera">
-        <pose> 0 0 0 0 0 0 </pose>
-        <visualize>true</visualize>
-        <update_rate>10</update_rate>
-        <camera>
-            <horizontal_fov>1.089</horizontal_fov>
-            <image>
-                <format>R8G8B8</format>
-                <width>640</width>
-                <height>480</height>
-            </image>
-            <clip>
-                <near>0.05</near>
-                <far>8.0</far>
-            </clip>
-        </camera>
-        <plugin name="camera_controller" filename="libgazebo_ros_camera.so">
-            <frame_name>camera_link_optical</frame_name>
-        </plugin>
+    <sensor name="rgb_camera" type="camera">
+      <pose>0 0 0 0 0 0</pose>
+      <visualize>true</visualize>
+      <update_rate>10</update_rate>
+      <camera>
+        <horizontal_fov>1.089</horizontal_fov>
+        <image>
+          <format>R8G8B8</format>
+          <width>640</width>
+          <height>480</height>
+        </image>
+        <clip>
+          <near>0.05</near>
+          <far>8.0</far>
+        </clip>
+      </camera>
+      <plugin name="camera_controller" filename="libgazebo_ros_camera.so">
+        <frameName>camera_link_optical</frameName>
+        <alwaysOn>true</alwaysOn>
+        <updateRate>10.0</updateRate>
+        <cameraName>rgb_camera</cameraName>
+        <imageTopicName>image_raw</imageTopicName>
+        <cameraInfoTopicName>camera_info</cameraInfoTopicName>
+        <robotNamespace>/rgb</robotNamespace>
+      </plugin>
     </sensor>
-</gazebo>
-<joint name="depth_camera_joint" type="fixed">
-  <parent link="base"/>
-  <child link="depth_camera_link"/>
-  <origin xyz="0.305 0.1 0.08" rpy="0 0 0"/>
-</joint>
-<link name="depth_camera_link">
-  <visual>
-    <geometry>
-      <box size="0.010 0.03 0.03"/>
-    </geometry>
-    <material name="blue"/>
-  </visual>
-</link>
-<joint name="depth_camera_optical_joint" type="fixed">
-  <parent link="depth_camera_link"/>
-  <child link="depth_camera_link_optical"/>
-  <origin xyz="0 0 0" rpy="${-pi/2} 0 ${-pi/2}"/>
-</joint>
-<link name="depth_camera_link_optical"/>
-<gazebo reference="depth_camera_link">
-  <material>Gazebo/Blue</material>
-  <sensor name="depth_camera" type="depth">
-    <pose>0 0 0 0 0 0</pose>
-    <visualize>true</visualize>
-    <update_rate>10</update_rate>
-    <camera>
-      <horizontal_fov>1.047</horizontal_fov>
-      <image>
-        <format>R8G8B8</format>
-        <width>640</width>
-        <height>480</height>
-      </image>
-      <clip>
-        <near>0.05</near>
-        <far>8.0</far>
-      </clip>
-    </camera>
-    <plugin name="depth_camera_controller" filename="libgazebo_ros_depth_camera.so">
-      <frame_name>depth_camera_link_optical</frame_name>
-      <min_depth>0.05</min_depth>
-      <max_depth>8.0</max_depth>
-    </plugin>
-  </sensor>
-</gazebo>
+  </gazebo>
+  <!-- ======================= -->
+  <!-- DEPTH CAMERA -->
+  <!-- ======================= -->
+  <joint name="depth_camera_joint" type="fixed">
+    <parent link="base"/>
+    <child link="depth_camera_link"/>
+    <origin xyz="0.305 0.1 0.08" rpy="0 0 0"/>
+  </joint>
+  <link name="depth_camera_link">
+    <visual>
+      <geometry>
+        <box size="0.010 0.03 0.03"/>
+      </geometry>
+      <material name="blue"/>
+    </visual>
+  </link>
+  <joint name="depth_camera_optical_joint" type="fixed">
+    <parent link="depth_camera_link"/>
+    <child link="depth_camera_link_optical"/>
+    <origin xyz="0 0 0" rpy="${-pi/2} 0 ${-pi/2}"/>
+  </joint>
+  <link name="depth_camera_link_optical"/>
+  <gazebo reference="depth_camera_link">
+    <material>Gazebo/Blue</material>
+    <sensor name="depth_camera" type="depth">
+      <pose>0 0 0 0 0 0</pose>
+      <visualize>true</visualize>
+      <update_rate>10</update_rate>
+      <camera>
+        <horizontal_fov>1.047</horizontal_fov>
+        <image>
+          <format>R8G8B8</format>
+          <width>640</width>
+          <height>480</height>
+        </image>
+        <clip>
+          <near>0.05</near>
+          <far>8.0</far>
+        </clip>
+      </camera>
+      <plugin name="depth_camera_controller" filename="libgazebo_ros_depth_camera.so">
+        <frameName>depth_camera_link_optical</frameName>
+        <alwaysOn>true</alwaysOn>
+        <updateRate>10.0</updateRate>
+        <cameraName>depth_camera</cameraName>
+        <imageTopicName>depth/image_raw</imageTopicName>
+        <cameraInfoTopicName>depth/camera_info</cameraInfoTopicName>
+        <robotNamespace>/depth</robotNamespace>
+        <minDepth>0.05</minDepth>
+        <maxDepth>8.0</maxDepth>
+      </plugin>
+    </sensor>
+  </gazebo>
 </robot>

Commit message: Replace camera and depth camera definitions with xacro:kinetic_rgb for improved sensor integration

File: sawyer_description/urdf/sawyer.urdf.xacro (robot description, xacro)
@@ -22,89 +22,8 @@
   </xacro:include>
   </xacro:if>
-  <joint name="camera_joint" type="fixed">
-    <parent link="base"/>
-    <child link="camera_link"/>
-    <origin xyz="0.305 0 0.08" rpy="0 0 0"/>
-</joint>
-<link name="camera_link">
-    <visual>
-        <geometry>
-            <box size="0.010 0.03 0.03"/>
-        </geometry>
-        <material name="red"/>
-    </visual>
-</link>
-<joint name="camera_optical_joint" type="fixed">
-    <parent link="camera_link"/>
-    <child link="camera_link_optical"/>
-    <origin xyz="0 0 0" rpy="${-pi/2} 0 ${-pi/2}"/>
-</joint>
-<link name="camera_link_optical"></link>
-<gazebo reference="camera_link">
-    <material>Gazebo/Red</material>
-    <sensor name="camera" type="camera">
-        <pose> 0 0 0 0 0 0 </pose>
-        <visualize>true</visualize>
-        <update_rate>10</update_rate>
-        <camera>
-            <horizontal_fov>1.089</horizontal_fov>
-            <image>
-                <format>R8G8B8</format>
-                <width>640</width>
-                <height>480</height>
-            </image>
-            <clip>
-                <near>0.05</near>
-                <far>8.0</far>
-            </clip>
-        </camera>
-        <plugin name="camera_controller" filename="libgazebo_ros_camera.so">
-            <frame_name>camera_link_optical</frame_name>
-        </plugin>
-    </sensor>
-</gazebo>
-<joint name="depth_camera_joint" type="fixed">
-  <parent link="base"/>
-  <child link="depth_camera_link"/>
-  <origin xyz="0.305 0.1 0.08" rpy="0 0 0"/>
-</joint>
-<link name="depth_camera_link">
-  <visual>
-    <geometry>
-      <box size="0.010 0.03 0.03"/>
-    </geometry>
-    <material name="blue"/>
-  </visual>
-</link>
-<joint name="depth_camera_optical_joint" type="fixed">
-  <parent link="depth_camera_link"/>
-  <child link="depth_camera_link_optical"/>
-  <origin xyz="0 0 0" rpy="${-pi/2} 0 ${-pi/2}"/>
-</joint>
-<link name="depth_camera_link_optical"/>
-<gazebo reference="depth_camera_link">
-  <material>Gazebo/Blue</material>
-  <sensor name="depth_camera" type="depth">
-    <pose>0 0 0 0 0 0</pose>
-    <visualize>true</visualize>
-    <update_rate>10</update_rate>
-    <camera>
-      <horizontal_fov>1.047</horizontal_fov>
-      <image>
-        <format>R8G8B8</format>
-        <width>640</width>
-        <height>480</height>
-      </image>
-      <clip>
-        <near>0.05</near>
-        <far>8.0</far>
-      </clip>
-    </camera>
-    <plugin name="depth_camera_controller" filename="libgazebo_ros_depth_camera.so">
-      <frame_name>depth_camera_link_optical</frame_name>
-      <min_depth>0.05</min_depth>
-      <max_depth>8.0</max_depth>
-    </plugin>
-  </sensor>
-</gazebo>
+  <xacro:include filename="$(find simulation)/urdf/sensors/kinetic_rgb.urdf.xacro"/>
+  <xacro:kinetic_rgb name="kinect" parent="base">
+    <origin xyz="0.5 0.0 1.0" rpy="0 1.57 0"/>
+    <optical_origin xyz="0 0 0" rpy="0 0 0"/>
+  </xacro:kinetic_rgb>
 </robot>

Commit message: Add additional RGB camera configurations to URDF

File: sawyer_description/urdf/sawyer.urdf.xacro (robot description, xacro)
@@ -5,7 +5,4 @@
   <xacro:arg name="static" default="true"/>
   <xacro:arg name="electric_gripper" default="false"/>
-  <!-- ======================= -->
-  <!-- SAWYER BASE -->
-  <!-- ======================= -->
   <xacro:include filename="$(find sawyer_description)/urdf/sawyer_base.urdf.xacro">
     <xacro:arg name="gazebo" value="${gazebo}"/>
@@ -24,7 +21,11 @@
   </xacro:if>
   <xacro:include filename="$(find simulation)/urdf/sensors/kinetic_rgb.urdf.xacro"/>
-  <xacro:kinetic_rgb name="kinect" parent="base">
+  <xacro:kinetic_rgb name="asus" parent="base">
     <origin xyz="0.5 0.0 1.0" rpy="0 1.57 0"/>
     <optical_origin xyz="0 0 0" rpy="0 0 0"/>
   </xacro:kinetic_rgb>
+  <xacro:kinetic_rgb name="logi" parent="base">
+    <origin xyz="1.5 0.0 1.0" rpy="0 1.57 0"/>
+    <optical_origin xyz="0 0 0" rpy="0 0 0"/>
+  </xacro:kinetic_rgb>
 </robot>

Commit message: Remove camera and depth camera configurations from URDF

File: sawyer_description/urdf/sawyer.urdf.xacro (robot description, xacro)
@@ -22,89 +22,3 @@
   </xacro:include>
   </xacro:if>
-  <joint name="camera_joint" type="fixed">
-    <parent link="base"/>
-    <child link="camera_link"/>
-    <origin xyz="0.305 0 0.08" rpy="0 0 0"/>
-</joint>
-<link name="camera_link">
-    <visual>
-        <geometry>
-            <box size="0.010 0.03 0.03"/>
-        </geometry>
-        <material name="red"/>
-    </visual>
-</link>
-<joint name="camera_optical_joint" type="fixed">
-    <parent link="camera_link"/>
-    <child link="camera_link_optical"/>
-    <origin xyz="0 0 0" rpy="${-pi/2} 0 ${-pi/2}"/>
-</joint>
-<link name="camera_link_optical"></link>
-<gazebo reference="camera_link">
-    <material>Gazebo/Red</material>
-    <sensor name="camera" type="camera">
-        <pose> 0 0 0 0 0 0 </pose>
-        <visualize>true</visualize>
-        <update_rate>10</update_rate>
-        <camera>
-            <horizontal_fov>1.089</horizontal_fov>
-            <image>
-                <format>R8G8B8</format>
-                <width>640</width>
-                <height>480</height>
-            </image>
-            <clip>
-                <near>0.05</near>
-                <far>8.0</far>
-            </clip>
-        </camera>
-        <plugin name="camera_controller" filename="libgazebo_ros_camera.so">
-            <frame_name>camera_link_optical</frame_name>
-        </plugin>
-    </sensor>
-</gazebo>
-<joint name="depth_camera_joint" type="fixed">
-  <parent link="base"/>
-  <child link="depth_camera_link"/>
-  <origin xyz="0.305 0.1 0.08" rpy="0 0 0"/>
-</joint>
-<link name="depth_camera_link">
-  <visual>
-    <geometry>
-      <box size="0.010 0.03 0.03"/>
-    </geometry>
-    <material name="blue"/>
-  </visual>
-</link>
-<joint name="depth_camera_optical_joint" type="fixed">
-  <parent link="depth_camera_link"/>
-  <child link="depth_camera_link_optical"/>
-  <origin xyz="0 0 0" rpy="${-pi/2} 0 ${-pi/2}"/>
-</joint>
-<link name="depth_camera_link_optical"/>
-<gazebo reference="depth_camera_link">
-  <material>Gazebo/Blue</material>
-  <sensor name="depth_camera" type="depth">
-    <pose>0 0 0 0 0 0</pose>
-    <visualize>true</visualize>
-    <update_rate>10</update_rate>
-    <camera>
-      <horizontal_fov>1.047</horizontal_fov>
-      <image>
-        <format>R8G8B8</format>
-        <width>640</width>
-        <height>480</height>
-      </image>
-      <clip>
-        <near>0.05</near>
-        <far>8.0</far>
-      </clip>
-    </camera>
-    <plugin name="depth_camera_controller" filename="libgazebo_ros_depth_camera.so">
-      <frame_name>depth_camera_link_optical</frame_name>
-      <min_depth>0.05</min_depth>
-      <max_depth>8.0</max_depth>
-    </plugin>
-  </sensor>
-</gazebo>
 </robot>

Commit message: Remove redundant RGB camera definitions from URDF for cleaner configuration

File: sawyer_description/urdf/sawyer.urdf.xacro (robot description, xacro)
@@ -21,11 +21,3 @@
   </xacro:if>
   <xacro:include filename="$(find simulation)/urdf/sensors/kinetic_rgb.urdf.xacro"/>
-  <xacro:kinetic_rgb name="asus" parent="base">
-    <origin xyz="0.5 0.0 1.0" rpy="0 1.57 0"/>
-    <optical_origin xyz="0 0 0" rpy="0 0 0"/>
-  </xacro:kinetic_rgb>
-  <xacro:kinetic_rgb name="logi" parent="base">
-    <origin xyz="1.5 0.0 1.0" rpy="0 1.57 0"/>
-    <optical_origin xyz="0 0 0" rpy="0 0 0"/>
-  </xacro:kinetic_rgb>
 </robot>
